File: stm32f030board.sch (KiCad schematic (older format))
At the start: 31 parts, among them J1 Conn_02x02_Odd_Even, J2 Conn_01x08, J3 105017-0001, J4 Conn_01x08, SW1 KLS7-TS3608-5.0-180, SW2 KLS7-TS3608-5.0-180, U1 24LC00, U2 STM32F030F4Px, U3 74HC164D, U4 LP5907MFX-3.3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

Commit message: ver with smal through hole
Connections:
- net +3V3: now also J2.7 (Pin_7)
- no-connect marks 8 -> 7
Changed lines of the file:
@@
 Text Label 4550 4450 2    50   ~ 0
 Q0
-NoConn ~ 3300 4450
 NoConn ~ 4100 6650
 Wire Wire Line
@@
 Connection ~ 2550 7150
 $Comp
-L power:GND #PWR?
+L power:+3.3V #PWR0132
+U 1 1 5F42EB96
+P 3300 4450
+F 0 "#PWR0132" H 3300 4300 50  0001 C CNN
+F 1 "+3.3V" H 3315 4623 50  0000 C CNN
+F 2 "" H 3300 4450 50  0001 C CNN
+F 3 "" H 3300 4450 50  0001 C CNN
+	1    3300 4450
+	0    -1   1    0
+$EndComp
+$Comp
+L power:GND #PWR0131
 U 1 1 5F2A7237
 P 3300 4550
-F 0 "#PWR?" H 3300 4300 50  0001 C CNN
+F 0 "#PWR0131" H 3300 4300 50  0001 C CNN
 F 1 "GND" H 3305 4377 50  0000 C CNN
 F 2 "" H 3300 4550 50  0001 C CNN
