File: stm32f030board.kicad_pcb (KiCad board)
At the start: 2 copper layers, 45.2 x 31.5 mm, 31 parts, among them J1 Conn_02x02_Odd_Even, J2 Conn_01x08, J3 105017-0001, J4 Conn_01x08, SW1 KLS7-TS3608-5.0-180, SW2 KLS7-TS3608-5.0-180, U1 24LC00, U2 STM32F030F4Px, U3 74HC164D, U4 LP5907MFX-3.3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

Commit message: ver with smal through hole
Connections:
- J2 pad 7: Net-(J2-Pad7) -> +3V3
Routing:
- net +3V3: track 52.2 -> 54.5 mm

Commit message: release v1.2
Parts:
- moved C10 0.68 mm to (144.7, 85.1)
- moved D2 0.33 mm to (158.9, 85.2)
Routing:
- net GND: track 104.1 -> 79.7 mm
- net +3V3: track 54.5 -> 52.0 mm
Other:
- board text added: "@bahoo08"
